File: IOT/RS232.kicad_sch (KiCad schematic)
At the start: 18 parts, among them IC1 MAX3222EAP+, IC2 MAX3222EAP+, J15 RS232_1, J16 RS232_1

Commit message: started pcb
Parts:
- IC1, IC2: footprint Library:SOP65P778X199-20N -> Package_SO:TSSOP-20_4.4x5mm_P0.4mm
Changed lines of the file:
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@@
 			)
 		)
-		(property "Footprint" "Library:SOP65P778X199-20N"
+		(property "Footprint" "Package_SO:TSSOP-20_4.4x5mm_P0.4mm"
 			(at 85.09 131.75 0)
 			(hide yes)
@@
 			)
 		)
-		(property "Footprint" "Library:SOP65P778X199-20N"
+		(property "Footprint" "Package_SO:TSSOP-20_4.4x5mm_P0.4mm"
 			(at 182.88 133.02 0)
 			(hide yes)
