File: IOT/IoT.kicad_sch (KiCad schematic)
At the start: 70 parts, among them J1 USB_C_Receptacle_USB2.0_16P, J10 Program header, J11 Conn_01x08_Pin, J12 Micro_SD_Card_Det2, J13 Conn_01x08_Pin, J14 Flow sensor, J2 Conn_01x01_Pin, J3 Conn_01x04_Pin, J4 Conn_01x01_Pin, J5 Conn_01x02_Pin, J6 Conn_01x02_Pin, J7 Conn_01x01_Pin, J8 Conn_01x05_Pin, J9 Conn_01x03_Pin, SW1 SW_Push, SW2 SW_Push, SW3 SW_Push, SW4 SW_Push, SW5 SW_Push, U1 STM32F401RETx, Y1 HSE, Y2 32.768khz

Commit message: started pcb
Parts:
- removed TP4: TestPoint_Flag, TestPoint:TestPoint_Pad_2.0x2.0mm, symbol Connector:TestPoint_Flag
- removed Y1: HSE, Crystal:Crystal_SMD_5032-2Pin_5.0x3.2mm_HandSoldering, symbol Device:Crystal
- added Y1: 16MHz, Crystal:Crystal_SMD_Abracon_ABM8AIG-4Pin_3.2x2.5mm, symbol Device:Crystal_GND23
- C12, C13, C6: footprint Capacitor_SMD:CP_Elec_4x5.4 -> Capacitor_SMD:C_0805_2012Metric_Pad1.18x1.45mm_HandSolder
- C2, C3: value 18p -> 22p
- D17, D18: footprint Diode_SMD:Littelfuse_PolyZen-LS -> Diode_SMD:D_1206_3216Metric_Pad1.42x1.75mm_HandSolder
- D19, D20: footprint Diode_SMD:Nexperia_DSN1608-2_1.6x0.8mm -> Diode_SMD:D_1206_3216Metric_Pad1.42x1.75mm_HandSolder
- J10, J8: footprint Connector_PinSocket_2.54mm:PinSocket_1x05_P2.54mm_Horizontal -> Connector_PinSocket_2.54mm:PinSocket_1x05_P2.54mm_Vertical
- J11, J13: footprint Connector_PinSocket_2.54mm:PinSocket_1x08_P2.54mm_Horizontal -> Connector_PinSocket_2.54mm:PinSocket_1x08_P2.54mm_Vertical
- J14: footprint Package_SO:TSSOP-8_3x3mm_P0.65mm -> Connector_PinSocket_2.54mm:PinSocket_1x04_P2.54mm_Vertical
- J2, J4, J7: footprint Connector_PinSocket_2.54mm:PinSocket_1x01_P2.54mm_Horizontal -> Connector_PinSocket_2.54mm:PinSocket_1x01_P2.54mm_Vertical
- J3: footprint Connector_PinSocket_2.54mm:PinSocket_1x04_P2.54mm_Horizontal -> Connector_PinSocket_2.54mm:PinSocket_1x04_P2.54mm_Vertical
- J5, J6: footprint Connector_PinSocket_2.54mm:PinSocket_1x02_P2.54mm_Horizontal -> Connector_PinSocket_2.54mm:PinSocket_1x02_P2.54mm_Vertical
- J9: footprint Connector_PinSocket_2.54mm:PinSocket_1x03_P2.54mm_Horizontal -> Connector_PinSocket_2.54mm:PinSocket_1x03_P2.54mm_Vertical
- R1, R10, R11, R12, R13, R14, R15, R2, R3, R4, R5, R6, R7, R8, R9: footprint Resistor_SMD:R_0805_2012Metric_Pad1.20x1.40mm_HandSolder -> LED_SMD:LED_1206_3216Metric_Pad1.42x1.75mm_HandSolder
- SW1, SW2, SW3, SW4, SW5: footprint Button_Switch_SMD:Panasonic_EVQPUJ_EVQPUA -> Button_Switch_SMD:SW_DIP_SPSTx01_Slide_6.7x4.1mm_W6.73mm_P2.54mm_LowProfile_JPin
- TP1, TP2, TP3, TP5, TP6, TP7: footprint TestPoint:TestPoint_Pad_2.0x2.0mm -> Connector_Pin:Pin_D0.7mm_L6.5mm_W1.8mm_FlatFork
Connections:
- net GND: now also Y1.2 (G), Y1.4 (G)
- net at C2.2, U1.5 (PH0): now also Y1.1
- net at C3.2, U1.6 (PH1): now also Y1.3

Commit message: routed full pcb
Parts:
- removed J2, J4, J7: Conn_01x01_Pin, Connector_PinSocket_2.54mm:PinSocket_1x01_P2.54mm_Vertical, symbol Connector:Conn_01x01_Pin
- removed J5, J6: Conn_01x02_Pin, Connector_PinSocket_2.54mm:PinSocket_1x02_P2.54mm_Vertical, symbol Connector:Conn_01x02_Pin
- removed J8: Conn_01x05_Pin, Connector_PinSocket_2.54mm:PinSocket_1x05_P2.54mm_Vertical, symbol Connector:Conn_01x05_Pin
- removed J9: Conn_01x03_Pin, Connector_PinSocket_2.54mm:PinSocket_1x03_P2.54mm_Vertical, symbol Connector:Conn_01x03_Pin
- added H1, H2, H3, H4: MountingHole, MountingHole:MountingHole_5.3mm_M5_ISO14580, symbol Mechanical:MountingHole
- added J2: Conn_01x20_Pin, Connector_PinHeader_2.54mm:PinHeader_1x20_P2.54mm_Vertical, symbol Connector:Conn_01x20_Pin
- added J4: Conn_01x04_Pin, Connector_PinSocket_2.54mm:PinSocket_1x04_P2.54mm_Vertical, symbol Connector:Conn_01x04_Pin
- J1: footprint Connector_USB:USB_C_Receptacle_Amphenol_12401948E412A -> Connector_USB:USB_C_Receptacle_G-Switch_GT-USB-7010ASV
Connections:
- net +3V3: now also J3.1 (Pin_1), J3.2 (Pin_2), J3.3 (Pin_3), J3.4 (Pin_4)
- net GND: now also J4.1 (Pin_1), J4.2 (Pin_2), J4.3 (Pin_3), J4.4 (Pin_4)
- net PB1: now also U1.27 (PB1), J2.8 (Pin_8); no longer R1.1, SW1.1, U1.51 (PC10)
- net PB2: now also U1.28 (PB2), J2.9 (Pin_9); no longer R2.1, SW2.1, U1.52 (PC11)
- net PB3: now also U1.55 (PB3), J2.10 (Pin_10); no longer R3.1, SW3.1, U1.53 (PC12)
- net PB0: now reaches U1.26 (PB0)
- net PB0: now also J2.7 (Pin_7)
- net PB4: now reaches U1.56 (PB4)
- net PB4: now also J2.11 (Pin_11)
- net PA0: now reaches U1.14 (PA0)
- net PA0: now also J2.1 (Pin_1)
- net PA1: now reaches U1.15 (PA1)
- net PA1: now also J2.2 (Pin_2)
- net PC0: now reaches U1.8 (PC0)
- net PC0: now also J2.15 (Pin_15); no longer J3.1 (Pin_1)
- net PC1: now reaches U1.9 (PC1)
- net PC1: now also J2.16 (Pin_16); no longer J3.2 (Pin_2)
- net PC2: now reaches U1.10 (PC2)
- net PC2: now also J2.17 (Pin_17); no longer J3.3 (Pin_3)
- net PC3: now reaches U1.11 (PC3)
- net PC3: now also J2.18 (Pin_18); no longer J3.4 (Pin_4)
- net PC13: now reaches U1.2 (PC13)
- net PC13: now also J2.20 (Pin_20)
- net PA4: now reaches U1.20 (PA4)
- net PA4: now also J2.3 (Pin_3)
- net PC5: now reaches U1.25 (PC5)
- net PC5: now also J2.19 (Pin_19)
- net PB10: now reaches U1.29 (PB10)
- net PB10: now also J2.14 (Pin_14)
- net PA9: now reaches U1.42 (PA9)
- net PA9: now also J2.4 (Pin_4)
- net PA10: now reaches U1.43 (PA10)
- net PA10: now also J2.5 (Pin_5)
- net PA15: now reaches U1.50 (PA15)
- net PA15: now also J2.6 (Pin_6)
- net PWMBlanket: now reaches U1.54 (PD2)
- net BP8: now reaches U1.61 (PB8)
- net BP8: now also J2.12 (Pin_12)
- net PB9: now reaches U1.62 (PB9)
- net PB9: now also J2.13 (Pin_13)
- new net BUTT1: R1.1, SW1.1, U1.51 (PC10)
- new net BUTT2: R2.1, SW2.1, U1.52 (PC11)
- new net BUTT3: R3.1, SW3.1, U1.53 (PC12)
Other:
- sheet Power ports: added PWMBlanket; removed none
- moved on the sheet: D1, R7, R8

Commit message: added silkscreen and updated footprints
Parts:
- D1: footprint Diode_SMD:D_0805_2012Metric_Pad1.15x1.40mm_HandSolder -> Diode_SMD:Nexperia_CFP3_SOD-123W
- D17, D18: footprint Diode_SMD:D_1206_3216Metric_Pad1.42x1.75mm_HandSolder -> Diode_SMD:Nexperia_CFP3_SOD-123W
Changed lines of the file:
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@@
 			)
 		)
-		(property "Footprint" "Diode_SMD:D_1206_3216Metric_Pad1.42x1.75mm_HandSolder"
+		(property "Footprint" "Diode_SMD:Nexperia_CFP3_SOD-123W"
 			(at 200.66 149.86 0)
 			(hide yes)
@@
 			)
 		)
-		(property "Footprint" "Diode_SMD:D_0805_2012Metric_Pad1.15x1.40mm_HandSolder"
+		(property "Footprint" "Diode_SMD:Nexperia_CFP3_SOD-123W"
 			(at 118.11 36.83 0)
 			(hide yes)
@@
 			)
 		)
-		(property "Footprint" "Diode_SMD:D_1206_3216Metric_Pad1.42x1.75mm_HandSolder"
+		(property "Footprint" "Diode_SMD:Nexperia_CFP3_SOD-123W"
 			(at 204.47 149.86 0)
 			(hide yes)
